Commit message: Corrections for PullRequest #1

File: xacro/base_car_sonar.xacro (robot description, xacro)
@@ -4,11 +4,9 @@
   <xacro:property name="concept" value="car_sonar"/>
   <!-- Loading vehicle's specific macros -->
-  <xacro:include filename="$(find  gazebo_ros_sonar_plugin)/xacro/snippets_${concept}.xacro"/>
-  <xacro:include filename="$(find uuv_descriptions)/models/common/urdf/common.urdf.xacro"/>
-  <xacro:include filename="$(find uuv_sensor_ros_plugins)/urdf/sensor_snippets.xacro"/>
+  <xacro:include filename="$(find  foward_looking_gazebo_sonar)/xacro/snippets_${concept}.xacro"/>
   <!--
     Vehicle's parameters (remember to enter the model parameters below)
   -->
-  <xacro:property name="visual_mesh_file" value="file://$(find  gazebo_ros_sonar_plugin)/meshes/Body_${concept}.stl"/>
+  <xacro:property name="visual_mesh_file" value="file://$(find  foward_looking_gazebo_sonar)/meshes/Body_${concept}.stl"/>
   <!-- Loading the UUV simulator ROS plugin macros -->
   <xacro:property name="mass" value="1000"/>
@@ -17,5 +15,5 @@
   <xacro:property name="rho" value="1028"/>
   <!-- Vehicle macro -->
-  <xacro:macro name="mccr_base" params="namespace *gazebo">
+  <xacro:macro name="car_sonar_base" params="namespace *gazebo">
     <!-- Rigid body description of the base link -->
     <link name="${namespace}/base_link">
@@ -78,7 +76,7 @@
     <xacro:insert_block name="gazebo"/>
     <!-- Include the thruster modules -->
-    <xacro:include filename="$(find gazebo_ros_sonar_plugin)/xacro/actuators_car_sonar.xacro"/>
+    <xacro:include filename="$(find foward_looking_gazebo_sonar)/xacro/actuators_car_sonar.xacro"/>
     <!-- Include the sensor modules -->
-    <xacro:include filename="$(find gazebo_ros_sonar_plugin)/xacro/sensors_car_sonar.xacro"/>
+    <xacro:include filename="$(find foward_looking_gazebo_sonar)/xacro/sensors_car_sonar.xacro"/>
   </xacro:macro>
 </robot>

File: xacro/default_car_sonar.xacro (robot description, xacro)
@@ -1,4 +1,4 @@
 <?xml version="1.0"?>
-<robot xmlns:xacro="http://www.ros.org/wiki/xacro" name="mccr">
+<robot xmlns:xacro="http://www.ros.org/wiki/xacro" name="car_sonar">
   <xacro:arg name="debug" default="0"/>
   <xacro:arg name="namespace" default="car_sonar"/>
@@ -6,14 +6,14 @@
   <!-- -->
   <!-- Include the ROV macro file -->
-  <xacro:include filename="$(find gazebo_ros_sonar_plugin)/xacro/base_$(arg concept).xacro"/>
-  <xacro:include filename="$(find gazebo_ros_sonar_plugin)/xacro/gazebo_$(arg concept).xacro"/>
+  <xacro:include filename="$(find foward_looking_gazebo_sonar)/xacro/base_$(arg concept).xacro"/>
+  <xacro:include filename="$(find foward_looking_gazebo_sonar)/xacro/gazebo_$(arg concept).xacro"/>
   <!-- -->
-  <!-- Create the mccr -->
-  <xacro:mccr_base namespace="$(arg namespace)">
+  <!-- Create the car_sonar -->
+  <xacro:car_sonar_base namespace="$(arg namespace)">
     <!-- -->
     <!-- Gazebo -->
     <gazebo>
     </gazebo>
-  </xacro:mccr_base>
+  </xacro:car_sonar_base>
   <!-- -->
     <gazebo>
@@ -23,11 +23,3 @@
       </plugin>
     </gazebo>
-  <!-- <link name="world"/>
-  <joint name="$(arg namespace)/base_link_joint" type="revolute">
-    <limit upper="0" lower="0" effort="1000000" velocity="0" />
-    <origin xyz="1.5 2 3" rpy="${pi} ${pi/2} 0"/>
-    <axis xyz="0 1 0" />
-    <parent link="world" />
-    <child link="$(arg namespace)/base_link" />
-  </joint> -->
 </robot>

File: xacro/gazebo_car_sonar.xacro (robot description, xacro)
@@ -3,6 +3,7 @@
 <gazebo reference="car_sonar/test_link">
 <sensor name='FLSonar' type='camera'>
-    <plugin name="SonarVisual" filename="libfl_sonar_ros.so" >
+    <plugin name="SonarVisual" filename="FowardLookingGazeboSonar.so" >
         <topic>car_sonar/FLSonar</topic>
+        <debug>1</debug>
         <link_reference>car_sonar/test_link</link_reference>
         <horizontal_fov>${pi/2}</horizontal_fov>

File: xacro/sensors_car_sonar.xacro (robot description, xacro)
@@ -1,6 +1,3 @@
 <?xml version="1.0"?>
 <robot xmlns:xacro="http://www.ros.org/wiki/xacro">
-<xacro:default_camera namespace="${namespace}" parent_link="${namespace}/base_link" suffix="down">
-    <origin xyz="0 0 1 " rpy="0 ${pi/2} 0"/>
-  </xacro:default_camera>
 </robot>

File: xacro/snippets_car_sonar.xacro (robot description, xacro)
@@ -65,6 +65,4 @@
           <mu1 value="1"/>
           <mu2 value="1"/>
-          <!-- <minDepth value="0.000001"/> -->
-          <!-- <maxContacts value="1"/> -->
           <kp  value="${kp_wheel}" />
           <kd  value="${kd_wheel}" />
@@ -77,6 +75,4 @@
           <mu1 value="1"/>
           <mu2 value="1"/>
-          <!-- <minDepth value="0.000001"/> -->
-          <!-- <maxContacts value="1"/> -->
           <kp  value="${kp_wheel}" />
           <kd  value="${kd_wheel}" />
@@ -89,6 +85,4 @@
           <mu1 value="1"/>
           <mu2 value="1"/>
-          <!-- <minDepth value="0.000001"/> -->
-          <!-- <maxContacts value="1"/> -->
           <kp  value="${kp_wheel}" />
           <kd  value="${kd_wheel}" />
@@ -101,6 +95,4 @@
           <mu1 value="1"/>
           <mu2 value="1"/>
-          <!-- <minDepth value="0.000001"/> -->
-          <!-- <maxContacts value="1"/> -->
           <kp  value="${kp_wheel}" />
           <kd  value="${kd_wheel}" />

Commit message: Documentation and minor improvements

File: xacro/base_car_sonar.xacro (robot description, xacro)
@@ -53,10 +53,10 @@
         <inertia ixx="0.01" ixy="0.001" ixz="0.001" iyy="0.01" iyz="0.001" izz="0.01"/>
       </inertial>
-      <!-- <visual>
-        <origin xyz="0 0 0" rpy="0 0 0"/>
+      <visual>
+        <origin xyz="0 0 0" rpy="0 ${pi/2} 0"/>
         <geometry>
-          <box size="0.4 0.8 0.1"/>
+          <cylinder length="0.2" radius="0.1"/>
         </geometry>
-      </visual> -->
+      </visual>
       <collision>
         <origin xyz="0 0 0" rpy="0 0 0"/>

Commit message: Correction of typo foward - forward

File: xacro/base_car_sonar.xacro (robot description, xacro)
@@ -4,9 +4,9 @@
   <xacro:property name="concept" value="car_sonar"/>
   <!-- Loading vehicle's specific macros -->
-  <xacro:include filename="$(find  foward_looking_gazebo_sonar)/xacro/snippets_${concept}.xacro"/>
+  <xacro:include filename="$(find  forward_looking_gazebo_sonar)/xacro/snippets_${concept}.xacro"/>
   <!--
     Vehicle's parameters (remember to enter the model parameters below)
   -->
-  <xacro:property name="visual_mesh_file" value="file://$(find  foward_looking_gazebo_sonar)/meshes/Body_${concept}.stl"/>
+  <xacro:property name="visual_mesh_file" value="file://$(find  forward_looking_gazebo_sonar)/meshes/Body_${concept}.stl"/>
   <!-- Loading the UUV simulator ROS plugin macros -->
   <xacro:property name="mass" value="1000"/>
@@ -67,16 +67,16 @@
     </link>
     <joint name="${namespace}/test_joint" type="revolute">
-      <origin xyz="0 0 3" rpy="0 ${pi/2} ${pi/2}"/>
+      <origin xyz="0 0 0.5" rpy="0 0 0"/>
+      <axis xyz="0 0 1" />
       <parent link="${namespace}/base_link" />
       <child link="${namespace}/test_link" />
       <limit upper="0" lower="0" effort="0" velocity="0" />
-      <axis xyz="1 0 0"/>
     </joint>
     <!-- Set up hydrodynamic plugin given as input parameter -->
     <xacro:insert_block name="gazebo"/>
     <!-- Include the thruster modules -->
-    <xacro:include filename="$(find foward_looking_gazebo_sonar)/xacro/actuators_car_sonar.xacro"/>
+    <xacro:include filename="$(find forward_looking_gazebo_sonar)/xacro/actuators_car_sonar.xacro"/>
     <!-- Include the sensor modules -->
-    <xacro:include filename="$(find foward_looking_gazebo_sonar)/xacro/sensors_car_sonar.xacro"/>
+    <xacro:include filename="$(find forward_looking_gazebo_sonar)/xacro/sensors_car_sonar.xacro"/>
   </xacro:macro>
 </robot>

File: xacro/default_car_sonar.xacro (robot description, xacro)
@@ -6,6 +6,6 @@
   <!-- -->
   <!-- Include the ROV macro file -->
-  <xacro:include filename="$(find foward_looking_gazebo_sonar)/xacro/base_$(arg concept).xacro"/>
-  <xacro:include filename="$(find foward_looking_gazebo_sonar)/xacro/gazebo_$(arg concept).xacro"/>
+  <xacro:include filename="$(find forward_looking_gazebo_sonar)/xacro/base_$(arg concept).xacro"/>
+  <xacro:include filename="$(find forward_looking_gazebo_sonar)/xacro/gazebo_$(arg concept).xacro"/>
   <!-- -->
   <!-- Create the car_sonar -->

File: xacro/gazebo_car_sonar.xacro (robot description, xacro)
@@ -3,5 +3,5 @@
 <gazebo reference="car_sonar/test_link">
 <sensor name='FLSonar' type='camera'>
-    <plugin name="SonarVisual" filename="libFowardLookingGazeboSonar.so" >
+    <plugin name="SonarVisual" filename="libForwardLookingGazeboSonar.so" >
         <topic>car_sonar/FLSonar</topic>
         <debug>1</debug>
@@ -17,6 +17,6 @@
         </image>
         <clip>
-            <near>0.1</near>
-            <far>5</far>
+            <near>3</near>
+            <far>15</far>
         </clip>
         <noise>

Commit message: Modification of names gazebo_sonar to sonar_gazebo

File: xacro/base_car_sonar.xacro (robot description, xacro)
@@ -4,9 +4,9 @@
   <xacro:property name="concept" value="car_sonar"/>
   <!-- Loading vehicle's specific macros -->
-  <xacro:include filename="$(find  forward_looking_gazebo_sonar)/xacro/snippets_${concept}.xacro"/>
+  <xacro:include filename="$(find  forward_looking_sonar_gazebo)/xacro/snippets_${concept}.xacro"/>
   <!--
     Vehicle's parameters (remember to enter the model parameters below)
   -->
-  <xacro:property name="visual_mesh_file" value="file://$(find  forward_looking_gazebo_sonar)/meshes/Body_${concept}.stl"/>
+  <xacro:property name="visual_mesh_file" value="file://$(find  forward_looking_sonar_gazebo)/meshes/Body_${concept}.stl"/>
   <!-- Loading the UUV simulator ROS plugin macros -->
   <xacro:property name="mass" value="1000"/>
@@ -76,7 +76,7 @@
     <xacro:insert_block name="gazebo"/>
     <!-- Include the thruster modules -->
-    <xacro:include filename="$(find forward_looking_gazebo_sonar)/xacro/actuators_car_sonar.xacro"/>
+    <xacro:include filename="$(find forward_looking_sonar_gazebo)/xacro/actuators_car_sonar.xacro"/>
     <!-- Include the sensor modules -->
-    <xacro:include filename="$(find forward_looking_gazebo_sonar)/xacro/sensors_car_sonar.xacro"/>
+    <xacro:include filename="$(find forward_looking_sonar_gazebo)/xacro/sensors_car_sonar.xacro"/>
   </xacro:macro>
 </robot>

File: xacro/default_car_sonar.xacro (robot description, xacro)
@@ -6,6 +6,6 @@
   <!-- -->
   <!-- Include the ROV macro file -->
-  <xacro:include filename="$(find forward_looking_gazebo_sonar)/xacro/base_$(arg concept).xacro"/>
-  <xacro:include filename="$(find forward_looking_gazebo_sonar)/xacro/gazebo_$(arg concept).xacro"/>
+  <xacro:include filename="$(find forward_looking_sonar_gazebo)/xacro/base_$(arg concept).xacro"/>
+  <xacro:include filename="$(find forward_looking_sonar_gazebo)/xacro/gazebo_$(arg concept).xacro"/>
   <!-- -->
   <!-- Create the car_sonar -->

Commit message: Test image to verify sonar orientation

File: xacro/base_car_sonar.xacro (robot description, xacro)
@@ -16,4 +16,5 @@
   <!-- Vehicle macro -->
   <xacro:macro name="car_sonar_base" params="namespace *gazebo">
+    <link name="world"/>
     <!-- Rigid body description of the base link -->
     <link name="${namespace}/base_link">
@@ -73,4 +74,9 @@
       <limit upper="0" lower="0" effort="0" velocity="0" />
     </joint>
+    <joint name="${namespace}/fixed_joint" type="fixed">
+      <origin xyz="3.5 -1 5" rpy="0 ${1*pi/10} 0"/>
+      <parent link="world" />
+      <child link="${namespace}/base_link" />
+    </joint>
     <!-- Set up hydrodynamic plugin given as input parameter -->
     <xacro:insert_block name="gazebo"/>

File: xacro/gazebo_car_sonar.xacro (robot description, xacro)
@@ -18,5 +18,5 @@
         <clip>
             <near>3</near>
-            <far>15</far>
+            <far>10</far>
         </clip>
         <noise>

Commit message: Orientation correction of the sonar image

File: xacro/base_car_sonar.xacro (robot description, xacro)
@@ -16,5 +16,4 @@
   <!-- Vehicle macro -->
   <xacro:macro name="car_sonar_base" params="namespace *gazebo">
-    <link name="world"/>
     <!-- Rigid body description of the base link -->
     <link name="${namespace}/base_link">
@@ -74,9 +73,4 @@
       <limit upper="0" lower="0" effort="0" velocity="0" />
     </joint>
-    <joint name="${namespace}/fixed_joint" type="fixed">
-      <origin xyz="3.5 -1 5" rpy="0 ${1*pi/10} 0"/>
-      <parent link="world" />
-      <child link="${namespace}/base_link" />
-    </joint>
     <!-- Set up hydrodynamic plugin given as input parameter -->
     <xacro:insert_block name="gazebo"/>
